File: pikas-pcbs.kicad_pcb (KiCad board)
At the start: 2 copper layers, 24 parts, among them SW1 SW_Push, U1 ATmega32U4-AU, Y1 16MHz

Commit message: redo
Parts:
- C3: value 22pF -> 1uF
- C4, R1, R2: moved to B.Cu
- F1: value Polyfuse -> 500mA; moved to B.Cu
- R3: value R_Small -> 22; moved to B.Cu
- moved R4 113.9 mm to (149.2, 81.0)
- moved C5 93.4 mm to (156.0, 62.2)
- moved C1 92.5 mm to (150.5, 53.0)
- moved Y1 92.0 mm to (145.7, 53.0)
- moved C2 91.9 mm to (141.5, 53.0)
- moved C7 91.3 mm to (140.0, 77.6)
- moved U1 91.3 mm to (143.9, 68.6)
- moved C3 84.6 mm to (126.9, 66.2)
- moved C6 75.1 mm to (138.6, 58.5), turned to 0 degrees
- moved SW1 52.4 mm to (126.1, 79.9)
- moved C4 38.8 mm to (77.8, 63.2), turned to 270 degrees
- moved F1 37.4 mm to (121.4, 65.7), turned to 90 degrees
- moved D1 36.3 mm to (94.9, 54.0)
- moved D2 36.3 mm to (114.0, 53.2)
- moved D3 36.3 mm to (94.9, 73.0)
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Other:
- board outline added: 84.1 x 43.7 mm

Commit message: hotfix
Parts:
- USB1: moved to B.Cu
- moved R1 8.77 mm to (129.4, 54.1)
- moved R3 5.46 mm to (123.7, 54.2)
Routing:
- net D+: track 0.00 -> 7.61 mm
- net D-: track 0.00 -> 7.54 mm
Other:
- net class Default: trace_width 0.25 -> 0.254
- net class Power added: clearance 0.2, trace_width 0.381, via_dia 0.8, via_drill 0.4
Changed lines of the file:
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@@
     (thickness 1.6)
     (drawings 8)
-    (tracks 0)
+    (tracks 7)
     (zones 0)
     (modules 24)
@@
   )
   (setup
-    (last_trace_width 0.25)
+    (last_trace_width 0.254)
     (trace_clearance 0.2)
     (zone_clearance 0.508)
@@
   (net_class Default "This is the default net class."
     (clearance 0.2)
-    (trace_width 0.25)
+    (trace_width 0.254)
     (via_dia 0.8)
     (via_drill 0.4)
     (uvia_dia 0.3)
     (uvia_drill 0.1)
-    (add_net +5V)
     (add_net D+)
     (add_net D-)
-    (add_net GND)
     (add_net "Net-(C3-Pad1)")
     (add_net "Net-(C4-Pad1)")
@@
     (add_net ROW0)
     (add_net ROW1)
+  )
+  (net_class Power ""
+    (clearance 0.2)
+    (trace_width 0.381)
+    (via_dia 0.8)
+    (via_drill 0.4)
+    (uvia_dia 0.3)
+    (uvia_drill 0.1)
+    (add_net +5V)
+    (add_net GND)
     (add_net VCC)
   )
@@
     )
   )
-  (module random-keyboard-parts:Molex-0548190589 (layer F.Cu)
+  (module random-keyboard-parts:Molex-0548190589 (layer B.Cu)
     (at 131.064 43.434 270)
     (attr smd)
-    (fp_text reference USB1 (at 2.032 0) (layer F.SilkS)
-      (effects (font (size 1 1) (thickness 0.15)))
+    (fp_text reference USB1 (at 2.032 0) (layer B.SilkS)
+      (effects (font (size 1 1) (thickness 0.15)) (justify mirror))
     )
     (fp_text value Molex-0548190589 (at -5.08 0) (layer Dwgs.User)
       (effects (font (size 1 1) (thickness 0.15)))
     )
-    (fp_text user %R (at 2 0) (layer F.CrtYd)
-      (effects (font (size 1 1) (thickness 0.15)))
-    )
-    (fp_line (start 3.25 -1.25) (end 5.5 -1.25) (layer F.CrtYd) (width 0.15))
-    (fp_line (start 5.5 -0.5) (end 3.25 -0.5) (layer F.CrtYd) (width 0.15))
-    (fp_line (start 3.25 0.5) (end 5.5 0.5) (layer F.CrtYd) (width 0.15))
-    (fp_line (start 5.5 1.25) (end 3.25 1.25) (layer F.CrtYd) (width 0.15))
-    (fp_line (start 3.25 2) (end 5.5 2) (layer F.CrtYd) (width 0.15))
-    (fp_line (start 3.25 -2) (end 3.25 2) (layer F.CrtYd) (width 0.15))
-    (fp_line (start 5.5 -2) (end 3.25 -2) (layer F.CrtYd) (width 0.15))
-    (fp_line (start -3.75 3.75) (end -3.75 -3.75) (layer F.CrtYd) (width 0.15))
-    (fp_line (start 5.5 3.75) (end -3.75 3.75) (layer F.CrtYd) (width 0.15))
-    (fp_line (start 5.5 -3.75) (end 5.5 3.75) (layer F.CrtYd) (width 0.15))
-    (fp_line (start -3.75 -3.75) (end 5.5 -3.75) (layer F.CrtYd) (width 0.15))
-    (fp_line (start 0 -3.85) (end 5.45 -3.85) (layer F.SilkS) (width 0.15))
-    (fp_line (start 0 3.85) (end 5.45 3.85) (layer F.SilkS) (width 0.15))
-    (fp_line (start 5.45 -3.85) (end 5.45 3.85) (layer F.SilkS) (width 0.15))
+    (fp_text user %R (at 2 0) (layer B.CrtYd)
+      (effects (font (size 1 1) (thickness 0.15)) (justify mirror))
+    )
+    (fp_line (start 3.25 1.25) (end 5.5 1.25) (layer B.CrtYd) (width 0.15))
+    (fp_line (start 5.5 0.5) (end 3.25 0.5) (layer B.CrtYd) (width 0.15))
+    (fp_line (start 3.25 -0.5) (end 5.5 -0.5) (layer B.CrtYd) (width 0.15))
+    (fp_line (start 5.5 -1.25) (end 3.25 -1.25) (layer B.CrtYd) (width 0.15))
+    (fp_line (start 3.25 -2) (end 5.5 -2) (layer B.CrtYd) (width 0.15))
+    (fp_line (start 3.25 2) (end 3.25 -2) (layer B.CrtYd) (width 0.15))
+    (fp_line (start 5.5 2) (end 3.25 2) (layer B.CrtYd) (width 0.15))
+    (fp_line (start -3.75 -3.75) (end -3.75 3.75) (layer B.CrtYd) (width 0.15))
+    (fp_line (start 5.5 -3.75) (end -3.75 -3.75) (layer B.CrtYd) (width 0.15))
+    (fp_line (start 5.5 3.75) (end 5.5 -3.75) (layer B.CrtYd) (width 0.15))
+    (fp_line (start -3.75 3.75) (end 5.5 3.75) (layer B.CrtYd) (width 0.15))
+    (fp_line (start 0 3.85) (end 5.45 3.85) (layer B.SilkS) (width 0.15))
+    (fp_line (start 0 -3.85) (end 5.45 -3.85) (layer B.SilkS) (width 0.15))
+    (fp_line (start 5.45 3.85) (end 5.45 -3.85) (layer B.SilkS) (width 0.15))
+    (fp_line (start -3.75 3.85) (end 0 3.85) (layer Dwgs.User) (width 0.15))
     (fp_line (start -3.75 -3.85) (end 0 -3.85) (layer Dwgs.User) (width 0.15))
-    (fp_line (start -3.75 3.85) (end 0 3.85) (layer Dwgs.User) (width 0.15))
-    (fp_line (start -1.75 -4.572) (end -1.75 4.572) (layer Dwgs.User) (width 0.15))
-    (fp_line (start -3.75 -3.85) (end -3.75 3.85) (layer Dwgs.User) (width 0.15))
+    (fp_line (start -1.75 4.572) (end -1.75 -4.572) (layer Dwgs.User) (width 0.15))
+    (fp_line (start -3.75 3.85) (end -3.75 -3.85) (layer Dwgs.User) (width 0.15))
+    (pad 6 thru_hole oval (at 0 3.65 270) (size 2.7 1.7) (drill oval 1.9 0.7) (layers *.Cu *.Mask)
+      (net 47 "Net-(USB1-Pad6)"))
     (pad 6 thru_hole oval (at 0 -3.65 270) (size 2.7 1.7) (drill oval 1.9 0.7) (layers *.Cu *.Mask)
       (net 47 "Net-(USB1-Pad6)"))
-    (pad 6 thru_hole oval (at 0 3.65 270) (size 2.7 1.7) (drill oval 1.9 0.7) (layers *.Cu *.Mask)
+    (pad 6 thru_hole oval (at 4.5 -3.65 270) (size 2.7 1.7) (drill oval 1.9 0.7) (layers *.Cu *.Mask)
       (net 47 "Net-(USB1-Pad6)"))
     (pad 6 thru_hole oval (at 4.5 3.65 270) (size 2.7 1.7) (drill oval 1.9 0.7) (layers *.Cu *.Mask)
       (net 47 "Net-(USB1-Pad6)"))
-    (pad 6 thru_hole oval (at 4.5 -3.65 270) (size 2.7 1.7) (drill oval 1.9 0.7) (layers *.Cu *.Mask)
-      (net 47 "Net-(USB1-Pad6)"))
-    (pad 5 smd rect (at 4.5 -1.6 270) (size 2.25 0.5) (layers F.Cu F.Paste F.Mask)
+    (pad 5 smd rect (at 4.5 1.6 270) (size 2.25 0.5) (layers B.Cu B.Paste B.Mask)
       (net 12 VCC))
-    (pad 4 smd rect (at 4.5 -0.8 270) (size 2.25 0.5) (layers F.Cu F.Paste F.Mask)
+    (pad 4 smd rect (at 4.5 0.8 270) (size 2.25 0.5) (layers B.Cu B.Paste B.Mask)
       (net 16 D-))
-    (pad 3 smd rect (at 4.5 0 270) (size 2.25 0.5) (layers F.Cu F.Paste F.Mask)
+    (pad 3 smd rect (at 4.5 0 270) (size 2.25 0.5) (layers B.Cu B.Paste B.Mask)
       (net 18 D+))
-    (pad 2 smd rect (at 4.5 0.8 270) (size 2.25 0.5) (layers F.Cu F.Paste F.Mask)
+    (pad 2 smd rect (at 4.5 -0.8 270) (size 2.25 0.5) (layers B.Cu B.Paste B.Mask)
       (net 48 "Net-(USB1-Pad2)"))
-    (pad 1 smd rect (at 4.5 1.6 270) (size 2.25 0.5) (layers F.Cu F.Paste F.Mask)
+    (pad 1 smd rect (at 4.5 -1.6 270) (size 2.25 0.5) (layers B.Cu B.Paste B.Mask)
       (net 1 GND))
   )
@@
   )
   (module Resistor_SMD:R_0805_2012Metric (layer B.Cu)
-    (at 129.159 54.0535 90)
+    (at 123.698 54.1505 90)
     (descr "Resistor SMD 0805 (2012 Metric), square (rectangular) end terminal, IPC_7351 nominal, (Body size source: https://docs.google.com/spreadsheets/d/1BsfQQcO9C6DZCsRaXUlFlo91Tg2WpOkGARC1WS5S8t0/edit?usp=sharing), generated with kicad-footprint-generator")
     (tags resistor)
@@
   )
   (module Resistor_SMD:R_0805_2012Metric (layer B.Cu)
-    (at 120.777 55.753 90)
+    (at 129.38125 54.0535 90)
     (descr "Resistor SMD 0805 (2012 Metric), square (rectangular) end terminal, IPC_7351 nominal, (Body size source: https://docs.google.com/spreadsheets/d/1BsfQQcO9C6DZCsRaXUlFlo91Tg2WpOkGARC1WS5S8t0/edit?usp=sharing), generated with kicad-footprint-generator")
     (tags resistor)
@@
   (gr_line (start 158.75 44.45) (end 158.75 81.75625) (layer Edge.Cuts) (width 0.05))
   (gr_line (start 77.7875 41.275) (end 155.575 41.275) (layer Edge.Cuts) (width 0.05))
+  (segment (start 129.937487 54.434763) (end 129.38125 54.991) (width 0.254) (layer B.Cu) (net 16))
+  (segment (start 130.40826 53.96399) (end 129.937487 54.434763) (width 0.254) (layer B.Cu) (net 16))
+  (segment (start 130.40826 49.45726) (end 130.40826 53.96399) (width 0.254) (layer B.Cu) (net 16))
+  (segment (start 130.264 49.313) (end 130.40826 49.45726) (width 0.254) (layer B.Cu) (net 16))
+  (segment (start 130.264 47.934) (end 130.264 49.313) (width 0.254) (layer B.Cu) (net 16))
+  (segment (start 131.064 53.564) (end 132.461 54.961) (width 0.254) (layer B.Cu) (net 18))
+  (segment (start 131.064 47.934) (end 131.064 53.564) (width 0.254) (layer B.Cu) (net 18))
 )

Commit message: SQUARE!!!
Parts:
- D1, D2, D3, D4: value D_Small -> SOD_123
- SW1: moved to B.Cu
- moved U1 47.3 mm to (96.9, 63.1), turned to 45 degrees
- moved C1 44.5 mm to (116.4, 81.5)
- moved C2 44.5 mm to (107.3, 81.6)
- moved Y1 44.5 mm to (111.6, 81.6)
- moved C5 38.3 mm to (118.3, 55.6), turned to 270 degrees
- moved R2 33.8 mm to (99.3, 47.7)
- moved R1 33.8 mm to (96.2, 47.7)
- moved USB1 33.6 mm to (97.6, 39.7)
- moved R4 31.3 mm to (118.3, 76.3)
- moved SW1 30.1 mm to (96.0, 81.8)
- moved C6 24.7 mm to (118.3, 44.5), turned to 270 degrees
- moved C7 22.4 mm to (118.3, 72.2), turned to 270 degrees
- moved C3 8.70 mm to (118.3, 67.5), turned to 270 degrees
- moved R3 6.83 mm to (118.3, 50.0), turned to 270 degrees
- moved F1 5.04 mm to (118.3, 61.7), turned to 270 degrees
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Routing:
- net D+: track 7.61 -> 0.00 mm
- net D-: track 7.54 -> 1.45 mm
- net Net-(R1-Pad2): track 0.00 -> 1.98 mm
Other:
- board size 84.1 x 43.7 mm -> 46.8 x 46.8 mm

Commit message: AWAITING LEON REVIEW BUT DONE
Parts:
- added ?: , , F.Cu at (118.9, 82.2)
- added REF**: MountingHole_2mm, MountingHole:MountingHole_2mm, F.Cu at (77.0, 82.3)
- added REF**: MountingHole_2mm, MountingHole:MountingHole_2mm, F.Cu at (118.9, 40.3)
- added REF**: MountingHole_2mm, MountingHole:MountingHole_2mm, F.Cu at (77.0, 40.3)
- moved C6 0.29 mm to (118.3, 44.7)
Routing:
- net GND: track 0.00 -> 188.5 mm, vias 0 -> 5
- net Net-(C3-Pad1): track 0.00 -> 96.6 mm, vias 0 -> 3
- net +5V: track 0.00 -> 93.3 mm, vias 0 -> 7
- net Net-(R3-Pad2): track 0.00 -> 66.2 mm, vias 0 -> 3
- net ROW0: track 0.00 -> 53.9 mm
- net Net-(C4-Pad1): track 0.00 -> 53.1 mm, vias 0 -> 2
- net Net-(C6-Pad1): track 0.00 -> 39.7 mm, vias 0 -> 2
- net VCC: track 0.00 -> 39.0 mm, vias 0 -> 2
- net Net-(R2-Pad2): track 0.00 -> 24.6 mm, vias 0 -> 4
- net Net-(R4-Pad2): track 0.00 -> 24.2 mm, vias 0 -> 2
- net Net-(MX3-Pad1): track 0.00 -> 23.7 mm
- net Net-(MX1-Pad1): track 0.00 -> 23.1 mm
- net Net-(R1-Pad2): track 1.98 -> 25.0 mm, vias 0 -> 2
- net Net-(D3-Pad2): track 0.00 -> 8.31 mm
- net Net-(D2-Pad2): track 0.00 -> 6.92 mm
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Other:
- net class Default removed
- net class Power removed
- board text added: "prod. toke"
